File: Linak-controller.kicad_pcb (KiCad board)
At the start: 4 copper layers, 125.8 x 100.6 mm, 48 parts, among them J1 Screw_Terminal_01x02, J2 Screw_Terminal_01x02, J4 Conn_02x03_Counter_Clockwise, J5 Screw_Terminal_01x02, J6 Screw_Terminal_01x02, J7 Screw_Terminal_01x02, K1 FINDER-36.11, K2 FINDER-36.11, K3 FINDER-36.11, K4 FINDER-36.11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

Commit message: fix some imperfections
Routing:
- net Relay_4_Polar_2: track 92.8 -> 91.8 mm
- net Relay_4_Polar_1: track 66.0 -> 65.4 mm
Changed lines of the file:
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@@
     (property "Sheetname" "")
     (attr smd)
-    (fp_text reference "R7" (at 0 -2.28) (layer "F.SilkS")
+    (fp_text reference "R7" (at -5.307 0.69) (layer "F.SilkS")
       (effects (font (size 1 1) (thickness 0.15)))
     )
@@
   (segment (start 26.416 56.388) (end 26.416 41.148) (width 1.02) (layer "F.Cu") (net 11))
   (segment (start 120.357 99.822) (end 115.666 104.513) (width 1.02) (layer "F.Cu") (net 11))
-  (segment (start 82.55 87.63) (end 35.306 87.63) (width 1.02) (layer "F.Cu") (net 12))
-  (segment (start 89.916 80.264) (end 82.55 87.63) (width 1.02) (layer "F.Cu") (net 12))
   (segment (start 113.284 86.614) (end 113.284 81.788) (width 1.02) (layer "F.Cu") (net 12))
+  (segment (start 33.782 92.549) (end 34.061 92.828) (width 1.02) (layer "F.Cu") (net 12))
+  (segment (start 33.782 90.932) (end 33.782 92.549) (width 1.02) (layer "F.Cu") (net 12))
   (segment (start 111.76 80.264) (end 89.916 80.264) (width 1.02) (layer "F.Cu") (net 12))
-  (segment (start 33.782 89.154) (end 33.782 92.549) (width 1.02) (layer "F.Cu") (net 12))
-  (segment (start 35.306 87.63) (end 33.782 89.154) (width 1.02) (layer "F.Cu") (net 12))
+  (segment (start 89.916 80.264) (end 81.788 88.392) (width 1.02) (layer "F.Cu") (net 12))
   (segment (start 113.284 81.788) (end 111.76 80.264) (width 1.02) (layer "F.Cu") (net 12))
+  (segment (start 81.788 88.392) (end 36.322 88.392) (width 1.02) (layer "F.Cu") (net 12))
+  (segment (start 36.322 88.392) (end 33.782 90.932) (width 1.02) (layer "F.Cu") (net 12))
   (segment (start 34.061 92.828) (end 33.646 92.828) (width 0.5) (layer "F.Cu") (net 12))
-  (segment (start 33.782 92.549) (end 34.061 92.828) (width 1.02) (layer "F.Cu") (net 12))
+  (segment (start 54.864 90.17) (end 90.678 90.17) (width 1.02) (layer "F.Cu") (net 13))
+  (segment (start 98.552 82.296) (end 109.474 82.296) (width 1.02) (layer "F.Cu") (net 13))
+  (segment (start 53.961 92.528) (end 53.961 91.073) (width 1.02) (layer "F.Cu") (net 13))
+  (segment (start 53.961 91.073) (end 54.864 90.17) (width 1.02) (layer "F.Cu") (net 13))
   (segment (start 109.474 82.296) (end 110.744 83.566) (width 1.02) (layer "F.Cu") (net 13))
-  (segment (start 83.566 89.154) (end 90.424 82.296) (width 1.02) (layer "F.Cu") (net 13))
-  (segment (start 90.424 82.296) (end 109.474 82.296) (width 1.02) (layer "F.Cu") (net 13))
-  (segment (start 53.961 92.528) (end 53.961 90.057) (width 1.02) (layer "F.Cu") (net 13))
+  (segment (start 90.678 90.17) (end 98.552 82.296) (width 1.02) (layer "F.Cu") (net 13))
   (segment (start 110.744 83.566) (end 110.744 86.614) (width 1.02) (layer "F.Cu") (net 13))
-  (segment (start 53.961 90.057) (end 54.864 89.154) (width 1.02) (layer "F.Cu") (net 13))
-  (segment (start 54.864 89.154) (end 83.566 89.154) (width 1.02) (layer "F.Cu") (net 13))
   (segment (start 93.218 51.562) (end 103.378 61.722) (width 1.02) (layer "F.Cu") (net 15))
   (segment (start 103.378 61.722) (end 119.126 61.722) (width 1.02) (layer "F.Cu") (net 15))
@@
         (xy 91.694 104.14)
         (xy 68.834 103.632)
-        (xy 64.008 121.158)
-        (xy 27.432 121.92)
-        (xy 27.686 91.44)
-        (xy 26.924 88.392)
-        (xy 26.162 69.85)
-        (xy 26.416 28.956)
-        (xy 36.83 29.21)
-        (xy 65.532 28.702)
-        (xy 69.088 44.958)
-        (xy 101.6 34.29)
+        (xy 64.262 119.888)
+        (xy 28.702 119.38)
+        (xy 28.448 91.186)
+        (xy 28.448 87.884)
+        (xy 28.194 69.342)
+        (xy 28.448 27.94)
+        (xy 36.83891 27.690654)
+        (xy 65.54091 28.198654)
+        (xy 66.548 42.926)
+        (xy 98.044 43.434)
         (xy 111.76 28.118965)
         (xy 136.144 27.94)
